File: headstage_hardware/analog.sch (KiCad schematic (older format))
At the start: 27 parts, among them U35 OMNETICS_36, U36 MIC5365-2.7, U37 TC1016-3.0, U39 9X100, U40 ADCS7476, U41 9X100, U45 RHA2132

Commit message: Started designing the headstage using 4 RHD2132 Intan chips. Need to interface with SPORTs instead of SPIs, like before.
Cleaned up some code.
Parts:
- C59, C60, C61, C62, C63, C64, C65, C66: symbol C -> C-RESCUE-stage9
- R67, R68, R69, R70, R71, R72, R73, R74, R75, R76, R77, R78: symbol R -> R-RESCUE-stage9

Commit message: Organized changes. Converted the old kicad projects. Started 4xRHD2132 headstage version. Recompiled gtkclient_multi for Ubuntu and newer protobufs.
Parts:
- C59, C60, C61, C62, C63, C64, C65, C66: symbol C-RESCUE-stage9 -> C
- R67, R68, R69, R70, R71, R72, R73, R74, R75, R76, R77, R78: symbol R-RESCUE-stage9 -> R
