File: headstage_hardware/analog.sch (KiCad schematic (older format))
At the start: 27 parts, among them U35 OMNETICS_36, U36 MIC5365-2.7, U37 TC1016-3.0, U39 9X100, U40 ADCS7476, U41 9X100, U45 RHA2132

Commit message: Screwed up the old kicad project files again by saving the board file. NEVER SAVE OLD .BRD FILES!!!
Fixed this and updated README with instructions to port old kicad
projects.
Parts:
- C59, C60, C61, C62, C63, C64, C65, C66: symbol C -> C-RESCUE-stage9
- R67, R68, R69, R70, R71, R72, R73, R74, R75, R76, R77, R78: symbol R -> R-RESCUE-stage9

Commit message: Fixed typos in headstage.cpp
Other:
- note added: "left of connector"
- note added: "right of connector"
Changed lines of the file:
@@
 $Descr User 16000 12000
 encoding utf-8
-Sheet 5 5
+Sheet 3 5
 Title "Stage 4 / Copyright 2010 Timothy L Hanson "
 Date "2 apr 2013"
@@
 	1    0    0    -1
 $EndComp
+Text Notes 2750 3950 0    60   ~ 0
+left of connector
+Text Notes 2650 5750 0    60   ~ 0
+right of connector
 $EndSCHEMATC
