File: headstage_hardware/stage9.sch (KiCad schematic (older format))
At the start: 65 parts, among them U1 VEE, U11 MAX6711Z, U12 ANTENNA, U3 9X100, U4 TPS62410, U46 9X100, U5 ABM10XTAL-16, U6 BF532-160, U8 NRF24L01, U9 SST25VF040B

Commit message: Started designing the headstage using 4 RHD2132 Intan chips. Need to interface with SPORTs instead of SPIs, like before.
Cleaned up some code.
Parts:
- C1, C10, C11, C12, C13, C14, C15, C16, C17, C18, C19, C2, C20, C21, C22, C23, C24, C25, C26, C27, C28, C29, C3, C30, C31, C32, C4, C6, C67, C68, C7, C8, C9: symbol C -> C-RESCUE-stage9
- D1: symbol LED -> LED-RESCUE-stage9
- R13, R14, R15, R16, R17, R21, R23, R26, R28, R29, R30, R79, R80, R81, R82: symbol R -> R-RESCUE-stage9

Commit message: Organized changes. Converted the old kicad projects. Started 4xRHD2132 headstage version. Recompiled gtkclient_multi for Ubuntu and newer protobufs.
Parts:
- C1, C10, C11, C12, C13, C14, C15, C16, C17, C18, C19, C2, C20, C21, C22, C23, C24, C25, C26, C27, C28, C29, C3, C30, C31, C32, C4, C6, C67, C68, C7, C8, C9: symbol C-RESCUE-stage9 -> C
- D1: symbol LED-RESCUE-stage9 -> LED
- R13, R14, R15, R16, R17, R21, R23, R26, R28, R29, R30, R79, R80, R81, R82: symbol R-RESCUE-stage9 -> R

Commit message: Screwed up the old kicad project files again by saving the board file. NEVER SAVE OLD .BRD FILES!!!
Fixed this and updated README with instructions to port old kicad
projects.
Parts:
- C1, C10, C11, C12, C13, C14, C15, C16, C17, C18, C19, C2, C20, C21, C22, C23, C24, C25, C26, C27, C28, C29, C3, C30, C31, C32, C4, C6, C67, C68, C7, C8, C9: symbol C -> C-RESCUE-stage9
- D1: symbol LED -> LED-RESCUE-stage9
- R13, R14, R15, R16, R17, R21, R23, R26, R28, R29, R30, R79, R80, R81, R82: symbol R -> R-RESCUE-stage9
