File: headstage2_hardware/headstage2.sch (KiCad schematic (older format))
At the start: 113 parts, among them U1 OMNETICS_A79025, U10 TPS62410, U11 ABM10XTAL, U12 BF532-160, U13 NRF24L01, U14 MAX6711T, U15 SST25VF040B, U16 9x100, U17 ANTENNA, U18 9x100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

Commit message: Fixed typos in headstage.cpp
Other:
- note added: "left of connector"
- note added: "right of connector"
Changed lines of the file:
@@
 Wire Wire Line
 	11125 3425 11125 3825
+Text Notes 1075 3800 0    60   ~ 0
+left of connector
+Text Notes 1025 1925 0    60   ~ 0
+right of connector
 $EndSCHEMATC
